File: pcb/memory_subsystem/control_logic.kicad_sch (KiCad schematic)
At the start: 6 parts, among them U22 74LS32, U23 74LS279, U24 74LS14

Commit message: Fixed spacing problem: no warnings/erros
Parts:
- added unit 3 of U24
- added unit 2 of U24
- renumbered U23 to U22, U22 to U23
Connections:
- no-connect marks 14 -> 18
Other:
- moved on the sheet: U22A, U22B, U22C, U22D, U23A

Commit message: Tracks finished
Parts:
- C22, C23, C24: footprint Capacitor_SMD:C_0805_2012Metric -> Capacitor_SMD:C_0805_2012Metric_Pad1.18x1.45mm_HandSolder
Changed lines of the file:
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@@
 			)
 		)
-		(property "Footprint" "Capacitor_SMD:C_0805_2012Metric"
+		(property "Footprint" "Capacitor_SMD:C_0805_2012Metric_Pad1.18x1.45mm_HandSolder"
 			(at 147.32 18.0848 0)
 			(hide yes)
@@
 			)
 		)
-		(property "Footprint" "Capacitor_SMD:C_0805_2012Metric"
+		(property "Footprint" "Capacitor_SMD:C_0805_2012Metric_Pad1.18x1.45mm_HandSolder"
 			(at 106.68 18.0848 0)
 			(hide yes)
@@
 			)
 		)
-		(property "Footprint" "Capacitor_SMD:C_0805_2012Metric"
+		(property "Footprint" "Capacitor_SMD:C_0805_2012Metric_Pad1.18x1.45mm_HandSolder"
 			(at 127 18.0848 0)
 			(hide yes)
